File: AVRx2_PCB/Thermocouple_Board_AVRx2.kicad_pcb (KiCad board)
At the start: 2 copper layers, 90 x 39 mm, 103 parts, among them J1 DAC_OUT, J2 SPI, J3 RST, J4 DAC, J5 UPDI-0, J6 UPDI-1, J7 EXP, Q1 DMN2310U, U1 AVR16EB, U10 MCP4726A0T-E/CH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

Commit message: Fix Typo
Other:
- board text added: "Https://github.com/Robherc/Thermocouple_Board"
- board text removed: "Https://github.com/Robherc/ThermocoupleBoard"
Changed lines of the file:
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@@
   (gr_line (start 194 78) (end 198 82)
     (stroke (width 0.05) (type default)) (layer "Edge.Cuts"))
-  (gr_text "Https://github.com/Robherc/ThermocoupleBoard" (at 170 109.75) (layer "B.SilkS")
+  (gr_text "Https://github.com/Robherc/Thermocouple_Board" (at 170 109.75) (layer "B.SilkS")
     (effects (font (size 1.25 1) (thickness 0.15)) (justify left bottom mirror))
   )
