File: AVRx2_PCB/Thermocouple_Board_AVRx2.kicad_pcb (KiCad board)
At the start: 2 copper layers, 90 x 39 mm, 103 parts, among them J1 DAC_OUT, J2 SPI, J3 RST, J4 DAC, J5 UPDI-0, J6 UPDI-1, J7 EXP, Q1 DMN2310U, U1 AVR16EB, U10 MCP4726A0T-E/CH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

Commit message: Fix crossed traces that were found during prototype testing
Connections:
- U1 pad 1: /Output MCU/CS -> Net-(U1-PC3)
- U1 pad 5: Net-(U1-PC3) -> /Output MCU/CS
- U9 pad 6: Net-(U2-PB3) -> Net-(U2-PB2)
- U9 pad 7: Net-(U2-PB2) -> Net-(U2-PB3)
Routing:
- net /Output MCU/CS: track 9.31 -> 12.0 mm, vias 0 -> 2
- net Net-(U2-PB2): track 13.7 -> 11.2 mm, vias 2 -> 0
- net Net-(U1-PC3): track 6.69 -> 7.84 mm, vias 0 -> 2
- net Net-(U2-PB3): track 10.7 -> 11.2 mm
Changed lines of the file:
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@@
       (net 5 "GND2") (pinfunction "Gnd2") (pintype "power_in"))
     (pad "6" smd roundrect (at 2.475 0.635) (size 1.95 0.6) (layers "F.Cu" "F.Paste" "F.Mask") (roundrect_rratio 0.25)
-      (net 51 "Net-(U2-PB3)") (pinfunction "IOB2") (pintype "bidirectional"))
+      (net 52 "Net-(U2-PB2)") (pinfunction "IOB2") (pintype "bidirectional"))
     (pad "7" smd roundrect (at 2.475 -0.635) (size 1.95 0.6) (layers "F.Cu" "F.Paste" "F.Mask") (roundrect_rratio 0.25)
-      (net 52 "Net-(U2-PB2)") (pinfunction "IOA2") (pintype "bidirectional"))
+      (net 51 "Net-(U2-PB3)") (pinfunction "IOA2") (pintype "bidirectional"))
     (pad "8" smd roundrect (at 2.475 -1.905) (size 1.95 0.6) (layers "F.Cu" "F.Paste" "F.Mask") (roundrect_rratio 0.25)
       (net 6 "3V3-ISO") (pinfunction "Vcc2") (pintype "power_in"))
@@
       (stroke (width 0.0254) (type solid)) (layer "F.Fab"))
     (pad "1" smd rect (at -3.6322 -4.224909 45) (size 1.651 0.4318) (layers "F.Cu" "F.Paste" "F.Mask")
-      (net 11 "/Output MCU/CS") (pinfunction "PA7") (pintype "unspecified"))
+      (net 40 "Net-(U1-PC3)") (pinfunction "PA7") (pintype "unspecified"))
     (pad "2" smd rect (at -3.6322 -3.574923 45) (size 1.651 0.4318) (layers "F.Cu" "F.Paste" "F.Mask")
       (net 12 "/Output MCU/MOSI") (pinfunction "PC0") (pintype "unspecified"))
@@
       (net 14 "/Output MCU/SCK") (pinfunction "PC2") (pintype "unspecified"))
     (pad "5" smd rect (at -3.6322 -1.624965 45) (size 1.651 0.4318) (layers "F.Cu" "F.Paste" "F.Mask")
-      (net 40 "Net-(U1-PC3)") (pinfunction "PC3") (pintype "unspecified"))
+      (net 11 "/Output MCU/CS") (pinfunction "PC3") (pintype "unspecified"))
     (pad "6" smd rect (at -3.6322 -0.974979 45) (size 1.651 0.4318) (layers "F.Cu" "F.Paste" "F.Mask")
       (net 15 "/Output MCU/DAC-High") (pinfunction "PD0") (pintype "unspecified"))
@@
   (segment (start 151.1 106.25) (end 151.1 104.9) (width 0.75) (layer "F.Cu") (net 9))
   (segment (start 164.85 99.5) (end 161.9625 99.5) (width 0.5) (layer "F.Cu") (net 10))
-  (segment (start 119.944185 99.580891) (end 119.919109 99.580891) (width 0.35) (layer "F.Cu") (net 11))
-  (segment (start 119.919109 99.580891) (end 118.06 101.44) (width 0.35) (layer "F.Cu") (net 11))
-  (segment (start 118.06 101.44) (end 111.4 101.44) (width 0.35) (layer "F.Cu") (net 11))
+  (segment (start 121.782623 101.419329) (end 121.780671 101.419329) (width 0.25) (layer "F.Cu") (net 11))
+  (segment (start 116 101.6) (end 114 101.6) (width 0.35) (layer "F.Cu") (net 11))
+  (segment (start 113.84 101.44) (end 111.4 101.44) (width 0.35) (layer "F.Cu") (net 11))
+  (segment (start 121.780671 101.419329) (end 120.4 102.8) (width 0.35) (layer "F.Cu") (net 11))
+  (segment (start 114 101.6) (end 113.84 101.44) (width 0.35) (layer "F.Cu") (net 11))
+  (via (at 116 101.6) (size 0.6) (drill 0.3) (layers "F.Cu" "B.Cu") (net 11))
+  (via (at 120.4 102.8) (size 0.6) (drill 0.3) (layers "F.Cu" "B.Cu") (net 11))
+  (segment (start 116.6 101) (end 116 101.6) (width 0.35) (layer "B.Cu") (net 11))
+  (segment (start 120.4 102.8) (end 118.6 101) (width 0.35) (layer "B.Cu") (net 11))
+  (segment (start 118.6 101) (end 116.6 101) (width 0.35) (layer "B.Cu") (net 11))
   (segment (start 115 102.5) (end 113.52 103.98) (width 0.35) (layer "F.Cu") (net 12))
   (segment (start 113.52 103.98) (end 111.4 103.98) (width 0.35) (layer "F.Cu") (net 12))
@@
   (segment (start 151.9 83.5) (end 151.9 81.6) (width 0.35) (layer "F.Cu") (net 39))
   (segment (start 151.9 81.6) (end 152.25 81.25) (width 0.35) (layer "F.Cu") (net 39))
-  (segment (start 121.782623 101.419329) (end 121.780671 101.419329) (width 0.25) (layer "F.Cu") (net 40))
   (segment (start 117.083363 106.116637) (end 117.083363 106.166637) (width 0.25) (layer "F.Cu") (net 40))
-  (segment (start 121.780671 101.419329) (end 117.083363 106.116637) (width 0.25) (layer "F.Cu") (net 40))
+  (segment (start 117.817705 101.682295) (end 119.919109 99.580891) (width 0.25) (layer "F.Cu") (net 40))
+  (segment (start 119.944185 99.580891) (end 119.919109 99.580891) (width 0.35) (layer "F.Cu") (net 40))
+  (segment (start 117.817705 101.742705) (end 117.817705 101.682295) (width 0.25) (layer "F.Cu") (net 40))
+  (segment (start 117.083363 106.166637) (end 117.825 105.425) (width 0.25) (layer "F.Cu") (net 40))
+  (via (at 117.817705 101.742705) (size 0.6) (drill 0.3) (layers "F.Cu" "B.Cu") (net 40))
+  (via (at 117.825 105.425) (size 0.6) (drill 0.3) (layers "F.Cu" "B.Cu") (net 40))
+  (segment (start 117.825 101.75) (end 117.825 105.425) (width 0.25) (layer "B.Cu") (net 40))
+  (segment (start 117.817705 101.742705) (end 117.825 101.75) (width 0.25) (layer "B.Cu") (net 40))
   (segment (start 120.73 105.22961) (end 120.73 106.945) (width 0.25) (layer "F.Cu") (net 41))
   (segment (start 123.161452 102.798158) (end 120.73 105.22961) (width 0.25) (layer "F.Cu") (net 41))
@@
   (segment (start 121.25 84) (end 121.25 82) (width 0.35) (layer "F.Cu") (net 50))
   (segment (start 128.625 90.625) (end 126.25 88.25) (width 0.35) (layer "F.Cu") (net 50))
-  (segment (start 161.525 93.54) (end 158.79 93.54) (width 0.5) (layer "F.Cu") (net 51))
-  (segment (start 154.885 89.635) (end 152.475 89.635) (width 0.5) (layer "F.Cu") (net 51))
-  (segment (start 158.79 93.54) (end 154.885 89.635) (width 0.5) (layer "F.Cu") (net 51))
-  (segment (start 156.25 92.75) (end 158.31 94.81) (width 0.5) (layer "F.Cu") (net 52))
-  (segment (start 156.25 92.5) (end 156.25 92.75) (width 0.5) (layer "F.Cu") (net 52))
-  (segment (start 158.31 94.81) (end 161.525 94.81) (width 0.5) (layer "F.Cu") (net 52))
-  (segment (start 155.25 88.365) (end 152.475 88.365) (width 0.5) (layer "F.Cu") (net 52))
-  (via (at 155.25 88.365) (size 0.8) (drill 0.4) (layers "F.Cu" "B.Cu") (net 52))
-  (via (at 156.25 92.5) (size 0.8) (drill 0.4) (layers "F.Cu" "B.Cu") (net 52))
-  (segment (start 155.25 91.5) (end 155.25 88.365) (width 0.5) (layer "B.Cu") (net 52))
-  (segment (start 156.25 92.5) (end 155.25 91.5) (width 0.5) (layer "B.Cu") (net 52))
+  (segment (start 154.115 88.365) (end 152.475 88.365) (width 0.5) (layer "F.Cu") (net 51))
+  (segment (start 155.385 89.635) (end 154.115 88.365) (width 0.5) (layer "F.Cu") (net 51))
+  (segment (start 161.525 93.54) (end 159.29 93.54) (width 0.5) (layer "F.Cu") (net 51))
+  (segment (start 159.29 93.54) (end 155.385 89.635) (width 0.5) (layer "F.Cu") (net 51))
+  (segment (start 159.21 94.81) (end 161.525 94.81) (width 0.5) (layer "F.Cu") (net 52))
+  (segment (start 152.475 89.635) (end 154.035 89.635) (width 0.5) (layer "F.Cu") (net 52))
+  (segment (start 154.035 89.635) (end 159.21 94.81) (width 0.5) (layer "F.Cu") (net 52))
   (segment (start 185.7 86.65) (end 187.1 86.65) (width 0.35) (layer "F.Cu") (net 53))
   (segment (start 188.741 100.882) (end 189.368 100.882) (width 0.25) (layer "F.Cu") (net 53))

Commit message: update to latest kicad version
Parts:
- L1: value 22uH -> SRF0703-6R8M
